File: Hardware/InkTime.sch (EAGLE design)
At the start: 105 parts, among them IC1 BQ25180YBGR, IC2 DRV2605YZFR, IC3 BMA423, IC9 RT6160AWSC, J1 503480-2400, J2 TC2030-IDC, J4 KH-TYPE-C-16P, Q1 20V/4.2A/52mΩ/1.4W, Q3 SI1308EDL-T1-GE3, U1 NRF52840_QF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

Commit message: Fixed #1. Added README.md, and updated the schematic and PCB design as stated in the issue.
Parts:
- C23, C27, C34, C42: device InkTime_v5:NORDIC_NRF_3_CAPACITOR_0201_L -> InkTime_v5:GRM011R60J152KE01L_2_GRM011R60J152KE01L
- C29, C30, C31, C32, C37, C38: device InkTime_v5:NORDIC_NRF_3_CAPACITOR_0402_L -> InkTime_v5:GRM011R60J152KE01L_2_GRM011R60J152KE01L
- EPD_C5: value 1uF/50V -> 0.1uF/50V; device InkTime_v5:NORDIC_NRF_3_CAPACITOR_0402_L -> InkTime_v5:NORDIC_NRF_3_CAPACITOR_0201_L
Connections:
- net GND: now also IC2.IN/TRIG; no longer IC2.SDA
- net SDA: now also IC2.SDA; no longer IC2.IN/TRIG
